File: AVR-Miner.kicad_pcb (KiCad board)
At the start: 2 copper layers, 20 x 30 mm, 15 parts, among them J1 Conn_01x04, J2 AVR-ISP-6, SW1 RESET, U1 ATmega328P-AU, Y1 16MHz

Commit message: Added v2.0.0
Parts:
- removed the G*** at (74.5, 43.5)
- removed the G*** at (86.5, 44.0)
- added G***: LOGO, MV_LOGO:MV_LOGO-8x5mm, B.Cu at (145.0, 91.3)
- added G***: LOGO, LOGO:BoardName, B.Cu at (145.0, 73.8)
- added G***: LOGO, MV_LOGO:maker.vinod-11x1.5mm, B.Cu at (145.0, 97.5)
- added JP1: Jumper_3_Open, Jumper:SolderJumper-3_P1.3mm_Open_RoundedPad1.0x1.5mm_NumberLabels, B.Cu at (151.5, 79.2)
- J1: value Conn_01x04 -> EXP; footprint Connector_PinHeader_2.54mm:PinHeader_1x04_P2.54mm_Vertical -> Connector_PinHeader_2.54mm:PinHeader_1x05_P2.54mm_Vertical
- moved R2 83.6 mm to (152.0, 77.0)
- moved U1 83.2 mm to (145.0, 86.5)
- moved Y1 83.2 mm to (145.0, 95.0)
- moved C1 83.2 mm to (152.0, 84.5)
- moved C2 83.2 mm to (138.0, 89.0)
- moved C3 83.2 mm to (137.8, 95.0)
- moved C4 83.2 mm to (152.2, 95.0)
- moved C5 83.2 mm to (152.0, 89.0)
- moved J2 83.2 mm to (142.5, 79.0)
- moved R1 83.2 mm to (138.0, 84.5)
- moved SW1 83.2 mm to (138.0, 77.5)
- moved D1 83.2 mm to (145.0, 73.5)
- moved J1 82.3 mm to (139.9, 100.0)
Connections:
- J1 pad 1: +5V -> EXT_LED
- J1 pad 2: SDA -> +5V
- J1 pad 3: SCL -> SDA
- J1 pad 4: GND -> SCL
- R2 pad 1: LED -> ON_BOARD_LED
Routing:
- net EXT_LED: track 0.00 -> 34.4 mm, vias 0 -> 1
- net ON_BOARD_LED: track 0.00 -> 2.90 mm, vias 0 -> 1
- net +5V: track 59.3 -> 60.0 mm
- net SCL: track 18.2 -> 18.7 mm
- net LED: track 12.5 -> 12.2 mm, vias 2 -> 1
Other:
- board text added: "LED"
- board text removed: "@maker.vinod"
- board text removed: "Duco-Miner"

Commit message: Updated project files for KiCad 7 & Added Gerber files
Connections:
- U1 pad 1: Net-(U1-Pad1) -> unconnected-(U1-PD3-Pad1)
- U1 pad 10: Net-(U1-Pad10) -> unconnected-(U1-PD6-Pad10)
- U1 pad 11: Net-(U1-Pad11) -> unconnected-(U1-PD7-Pad11)
- U1 pad 12: Net-(U1-Pad12) -> unconnected-(U1-PB0-Pad12)
- U1 pad 13: Net-(U1-Pad13) -> unconnected-(U1-PB1-Pad13)
- U1 pad 14: Net-(U1-Pad14) -> unconnected-(U1-PB2-Pad14)
- U1 pad 19: Net-(U1-Pad19) -> unconnected-(U1-ADC6-Pad19)
- U1 pad 2: Net-(U1-Pad2) -> unconnected-(U1-PD4-Pad2)
- U1 pad 22: Net-(U1-Pad22) -> unconnected-(U1-ADC7-Pad22)
- U1 pad 23: Net-(U1-Pad23) -> unconnected-(U1-PC0-Pad23)
- U1 pad 24: Net-(U1-Pad24) -> unconnected-(U1-PC1-Pad24)
- U1 pad 25: Net-(U1-Pad25) -> unconnected-(U1-PC2-Pad25)
- U1 pad 26: Net-(U1-Pad26) -> unconnected-(U1-PC3-Pad26)
- U1 pad 30: Net-(U1-Pad30) -> unconnected-(U1-PD0-Pad30)
- U1 pad 31: Net-(U1-Pad31) -> unconnected-(U1-PD1-Pad31)
- U1 pad 32: Net-(U1-Pad32) -> unconnected-(U1-PD2-Pad32)
- U1 pad 9: Net-(U1-Pad9) -> unconnected-(U1-PD5-Pad9)
Other:
- net class Default removed
